Commit message: First commit

File: rbpodo_description/robots/rb10_1300e.urdf (copy).xacro (robot description, xacro)
@@ -4,5 +4,4 @@
   <xacro:include filename="$(find rbpodo_description)/robots/rb_6dof.xacro" />
   <xacro:include filename="$(find rbpodo_description)/robots/rb_6dof.ros2_control.xacro" />
-  <xacro:include filename="$(find rbpodo_description)/robots/sensors/tof_gpu_lidar.xacro"/>
   <!-- ================= Arguments ================= -->
   <xacro:arg name="prefix" default="" />
@@ -31,67 +30,4 @@
       tcp_xyz="0 -0.1153 0"
       tcp_rpy="0 0 0" />
-      <!-- link2: RIGHT(+Y->-Y는 로봇 정의에 따라 다름, 여기선 방향만 예시) -->
-<!-- link2 ToFs -->
-<!-- =============================== -->
-<!-- Link-specific ToF base offsets -->
-<!-- =============================== -->
-<!-- link2 -->
-<xacro:property name="link2_tof_x" value="0.0"/>
-<xacro:property name="link2_tof_y" value="-0.1875"/>
-<xacro:property name="link2_tof_z" value="0.30635"/>
-<!-- link3 -->
-<xacro:property name="link3_tof_x" value="0.0"/>
-<xacro:property name="link3_tof_y" value="0.1484"/>
-<xacro:property name="link3_tof_z" value="0.285075"/>
-<!-- ================= link2 ToF ================= -->
-<xacro:tof_gpu_lidar
-  parent="link2"
-  name="link2_tof_north"
-  xyz="${link2_tof_x+0.075} ${link2_tof_y} ${link2_tof_z}"
-  rpy="0 0 0"
-  topic="/link2/tof_north"/>
-<xacro:tof_gpu_lidar
-  parent="link2"
-  name="link2_tof_south"
-  xyz="${link2_tof_x-0.075} ${link2_tof_y} ${link2_tof_z}"
-  rpy="0 0 3.14159"
-  topic="/link2/tof_south"/>
-<xacro:tof_gpu_lidar
-  parent="link2"
-  name="link2_tof_west"
-  xyz="${link2_tof_x} ${link2_tof_y+0.075} ${link2_tof_z}"
-  rpy="0 0 1.5708"
-  topic="/link2/tof_west"/>
-<xacro:tof_gpu_lidar
-  parent="link2"
-  name="link2_tof_east"
-  xyz="${link2_tof_x} ${link2_tof_y-0.075} ${link2_tof_z}"
-  rpy="0 0 -1.5708"
-  topic="/link2/tof_east"/>
-<!-- ================= link3 ToF ================= -->
-<xacro:tof_gpu_lidar
-  parent="link3"
-  name="link3_tof_north"
-  xyz="${link3_tof_x+0.06} ${link3_tof_y} ${link3_tof_z}"
-  rpy="0 0 0"
-  topic="/link3/tof_north"/>
-<xacro:tof_gpu_lidar
-  parent="link3"
-  name="link3_tof_south"
-  xyz="${link3_tof_x-0.06} ${link3_tof_y} ${link3_tof_z}"
-  rpy="0 0 3.14159"
-  topic="/link3/tof_south"/>
-<xacro:tof_gpu_lidar
-  parent="link3"
-  name="link3_tof_west"
-  xyz="${link3_tof_x} ${link3_tof_y+0.06} ${link3_tof_z}"
-  rpy="0 0 1.5708"
-  topic="/link3/tof_west"/>
-<xacro:tof_gpu_lidar
-  parent="link3"
-  name="link3_tof_east"
-  xyz="${link3_tof_x} ${link3_tof_y-0.06} ${link3_tof_z}"
-  rpy="0 0 -1.5708"
-  topic="/link3/tof_east"/>
   <!-- ================= ros2_control ================= -->
   <xacro:rb_6dof_ros2_control

File: rbpodo_description/robots/rb_6dof.ros2_control.xacro (robot description, xacro)
@@ -1,35 +1,47 @@
 <?xml version='1.0' encoding='utf-8'?>
 <robot xmlns:xacro="http://www.ros.org/wiki/xacro">
-  <xacro:macro name="rb_6dof_ros2_control" params="prefix robot_ip cb_simulation:=^|false use_fake_hardware:=^|false fake_sensor_commands:=^|false torque_constants:=${[1, 1, 1, 1, 1, 1]}">
+  <xacro:macro name="rb_6dof_ros2_control" params="prefix robot_ip cb_simulation use_fake_hardware fake_sensor_commands torque_constants">
     <ros2_control name="RBPodoHardwareInterface" type="system">
       <hardware>
-        <xacro:if value="${use_fake_hardware}">
-          <plugin>mock_components/GenericSystem</plugin>
-          <param name="mock_sensor_commands">${fake_sensor_commands}</param>
-          <param name="state_following_offset">0.0</param>
-        </xacro:if>
-        <xacro:unless value="${use_fake_hardware}">
-          <plugin>rbpodo_hardware/RBPodoHardwareInterface</plugin>
-          <param name="cb_simulation">${cb_simulation}</param>
-          <param name="robot_ip">${robot_ip}</param>
-        </xacro:unless>
+        <plugin>gz_ros2_control/GazeboSimSystem</plugin>
+         <param name="position_proportional_gain">20.0</param>
+         <param name="position_derivative_gain">2.0</param>
       </hardware>
-      <xacro:macro name="configure_joint" params="joint_name torque_constant:=1">
-        <joint name="${joint_name}">
-          <param name="initial_position">0.0</param>
-          <param name="torque_constant">${torque_constant}</param>
-          <command_interface name="effort"/>
-          <command_interface name="velocity"/>
-          <command_interface name="position"/>
-          <state_interface name="position"/>
-          <state_interface name="effort"/>
-        </joint>
-      </xacro:macro>
-      <xacro:configure_joint joint_name="${prefix}base" torque_constant="${torque_constants[0]}" />
-      <xacro:configure_joint joint_name="${prefix}shoulder" torque_constant="${torque_constants[1]}" />
-      <xacro:configure_joint joint_name="${prefix}elbow" torque_constant="${torque_constants[2]}" />
-      <xacro:configure_joint joint_name="${prefix}wrist1" torque_constant="${torque_constants[3]}" />
-      <xacro:configure_joint joint_name="${prefix}wrist2" torque_constant="${torque_constants[4]}" />
-      <xacro:configure_joint joint_name="${prefix}wrist3" torque_constant="${torque_constants[5]}" />
+      <joint name="${prefix}base">
+        <command_interface name="position"/>
+        <state_interface name="position"/>
+        <state_interface name="velocity"/>
+        <state_interface name="effort"/>
+      </joint>
+      <joint name="${prefix}shoulder">
+        <command_interface name="position"/>
+        <state_interface name="position"/>
+        <state_interface name="velocity"/>
+        <state_interface name="effort"/>
+      </joint>
+      <joint name="${prefix}elbow">
+        <command_interface name="position"/>
+        <state_interface name="position"/>
+        <state_interface name="velocity"/>
+        <state_interface name="effort"/>
+      </joint>
+      <joint name="${prefix}wrist1">
+        <command_interface name="position"/>
+        <state_interface name="position"/>
+        <state_interface name="velocity"/>
+        <state_interface name="effort"/>
+      </joint>
+      <joint name="${prefix}wrist2">
+        <command_interface name="position"/>
+        <state_interface name="position"/>
+        <state_interface name="velocity"/>
+        <state_interface name="effort"/>
+      </joint>
+      <joint name="${prefix}wrist3">
+        <command_interface name="position"/>
+        <state_interface name="position"/>
+        <state_interface name="velocity"/>
+        <state_interface name="effort"/>
+      </joint>
     </ros2_control>
   </xacro:macro>

File: rbpodo_description/robots/rb_6dof.xacro (robot description, xacro)
@@ -16,5 +16,4 @@
       </collision>
       <xacro:if value="${has_inertial}">
-        <!-- Check whether this property is available or not -->
         <xacro:property name="props" value="${links_props[name]}" />
         <xacro:property name="inertial" value="${props.inertial}" />
@@ -31,5 +30,4 @@
     <xacro:property name="joints_props_file" value="$(find rbpodo_description)/robots/${model_id}/joint.yaml" />
     <xacro:property name="joints_props" value="${xacro.load_yaml(joints_props_file)}" />
-    <!-- Check whether name is in joints_props or not -->
     <xacro:property name="props" value="${joints_props[name]}" />
     <joint name="${name}" type="revolute">
@@ -43,5 +41,21 @@
   </xacro:macro>
   <xacro:macro name="rb_6dof" params="model_id prefix='' tcp_name='tcp' tcp_xyz='0 0 0' tcp_rpy='0 0 0'">
-    <xacro:link name="${prefix}link0" has_inertial="false" />
+    <link name="${prefix}link0">
+      <visual>
+        <geometry>
+          <mesh filename="package://rbpodo_description/meshes/${model_id}/visual/link0.dae" />
+        </geometry>
+      </visual>
+      <collision>
+        <geometry>
+          <mesh filename="package://rbpodo_description/meshes/${model_id}/collision/link0.stl" />
+        </geometry>
+      </collision>
+      <inertial>
+        <origin xyz="0 0 0" rpy="0 0 0"/>
+        <mass value="5.0"/>
+        <inertia ixx="0.01" ixy="0.0" ixz="0.0" iyy="0.01" iyz="0.0" izz="0.01"/>
+      </inertial>
+    </link>
     <xacro:link name="${prefix}link1" />
     <xacro:link name="${prefix}link2" />
